File: InvitaciónTDS_robotica/InvitaciónTDS_general.kicad_pcb (KiCad board)
At the start: 2 copper layers, 95 x 95 mm, 38 parts, among them J1 Voltage Conn, J2 FTDI Connector, Q1 2N2219, Q2 2N2219, Q3 2N2219, Q4 2N2219, Q5 2N2219, Q6 2N2219, Q7 2N2219, SW1 SW_Push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

Commit message: update robotica
Parts:
- removed the G*** at (110.0, 135.0)
- removed J1: Voltage Conn, Connector_PinHeader_2.54mm:PinHeader_1x08_P2.54mm_Vertical
- A1: moved to B.Cu
- moved D5 174.5 mm to (72.0, 94.2)
- moved R5 164.1 mm to (70.8, 88.6)
- moved Q7 163.5 mm to (75.5, 130.3)
- moved D1 160.7 mm to (103.1, 83.2)
- moved Q5 158.6 mm to (78.3, 94.8)
- moved BZ2 151.0 mm to (79.4, 79.6)
- moved R1 149.4 mm to (104.6, 92.8)
- moved U1 144.2 mm to (95.4, 56.4)
- moved R9 142.2 mm to (71.7, 126.2), turned to 90 degrees
- moved Q1 141.9 mm to (111.6, 86.8)
- moved R7 139.9 mm to (75.1, 126.2), turned to 90 degrees
- moved C2 137.3 mm to (77.7, 107.2)
- moved D6 136.2 mm to (90.9, 95.8)
- moved R8 135.9 mm to (78.5, 126.2), turned to 90 degrees
- moved D3 135.7 mm to (132.7, 90.8)
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Other:
- outline, holes or cut-outs redrawn
- board text added: "06 Julio 2025"
- board text added: "ALEJANDRO GARCIA ANDRES RODRIGUEZ ARIADNA MEDINA ANGELA PAEZ CESAR BENAVIDES DANIEL SANCHEZ DANIEL CASTAÑON DAVID ISRAEL EMILIO RIZO EUGENIO TREVIÑO FRANCISCO FORTUNA JUAN PABLO JUAN CARLOS HERNANDEZ LUIZ ZERMEÑO MARCELO CUEVAS RODRIGO ESCANDON ALEXIS CHAPA DANITZA DEMIAN"
- board text added: "ROBÓTICA Y"
- board text added: "SISTEMAS DIGITALES"
- board text removed: "06 JULIO 2025"
- board text removed: "ELECTRÓNICA"

Commit message: terminado
Parts:
- removed BZ2: Buzzer, Buzzer_Beeper:Buzzer_12x9.5RM7.6
- removed D6: LED, LED_THT:LED_D5.0mm
- removed Q6: 2N2219, Package_TO_SOT_THT:TO-92_Inline
- removed R6: R, Resistor_THT:R_Axial_DIN0207_L6.3mm_D2.5mm_P10.16mm_Horizontal
- added G***: LOGO, LOGO, F.Cu at (109.5, 142.2)
- added G***: LOGO, LOGO, B.Cu at (80.0, 75.4)
- R2, R8: moved to B.Cu
- moved R9 98.5 mm to (141.9, 57.0), turned to 0 degrees
- moved R7 94.7 mm to (157.5, 79.5)
- moved C2 88.6 mm to (154.5, 63.0)
- moved MK1 87.6 mm to (146.3, 63.0)
- moved C1 85.9 mm to (151.0, 70.0), turned to 0 degrees
- moved R5 85.2 mm to (142.4, 134.8)
- moved Q7 83.4 mm to (145.7, 85.4)
- moved RV1 82.7 mm to (83.9, 55.4), turned to 90 degrees
- moved BZ1 80.5 mm to (76.5, 100.0), turned to 180 degrees
- moved G*** 76.5 mm to (82.0, 63.6)
- moved U2 71.1 mm to (77.8, 129.3), turned to 180 degrees
- moved Q5 69.8 mm to (135.5, 134.8)
- moved R8 69.2 mm to (139.0, 92.5)
- moved D5 68.3 mm to (127.0, 134.8)
- moved D2 66.9 mm to (152.5, 86.0)
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Routing:
- net GND: track 0.00 -> 273.8 mm, vias 0 -> 3
- net /LEDSchem/PinName: track 0.00 -> 220.3 mm
- net Net-(A1-+5V): track 0.00 -> 135.5 mm
- net Net-(A1-D2): track 0.00 -> 74.0 mm, vias 0 -> 2
- net Net-(A1-D0/RX): track 0.00 -> 51.9 mm, vias 0 -> 1
- net Net-(A1-D6): track 0.00 -> 51.5 mm
- net Net-(A1-D1/TX): track 0.00 -> 47.7 mm, vias 0 -> 1
- net Net-(Q7-C): track 0.00 -> 45.1 mm
- net Net-(A1-A0): track 0.00 -> 39.3 mm
- net /LEDSchem2/PinName: track 0.00 -> 39.2 mm
- net Net-(A1-A1): track 0.00 -> 38.7 mm
- net Net-(Q7-B): track 0.00 -> 27.3 mm
- net Net-(Q4-B): track 0.00 -> 18.0 mm
- net Net-(MK1-+): track 0.00 -> 16.8 mm
- net Net-(D1-K): track 0.00 -> 15.1 mm
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- added copper zone on B.Cu, net GND
- added copper zone on F.Cu, net GND
Other:
- outline, holes or cut-outs redrawn
- board text added: "06 JULIO 2025"
- board text added: "Alexis Chapa Andrés Carrizales Ángela Páez Ariadna Medina Eric González César Benavides Alejandro García Daniel Castañon Daniel Salinas Daniela Martínez David Vázquez Demian Marín"
- board text added: "Emilio Rizo Eugenio Treviño Francisco Velazquez Francisco Fortuna Jesús Gómez Jorge Molina José Tomé Emiliano Flores José Pablo Cedano Juan Carlos Hernández Julio Reséndiz Laura Méndez"
- board text added: "Luis Zermeño Mario Lozoya Manuel Sánchez Marcelo Cuevas Mario Cervantes Max Pacheco Neil Hernández Omar Flores Pamela Hernández Rodrigo Escandón Rodrigo Ibara Victor Vázquez Xóchitl Martínez"
- board text removed: "06 Julio 2025"
- board text removed: "ALEJANDRO GARCIA ANDRES RODRIGUEZ ARIADNA MEDINA ANGELA PAEZ CESAR BENAVIDES DANIEL SANCHEZ DANIEL CASTAÑON DAVID ISRAEL EMILIO RIZO EUGENIO TREVIÑO FRANCISCO FORTUNA JUAN PABLO JUAN CARLOS HERNANDEZ LUIZ ZERMEÑO MARCELO CUEVAS RODRIGO ESCANDON ALEXIS CHAPA DANITZA DEMIAN"
